Commit message: urdf, launch changes

File: my_bot/description/test_robot.urdf.xacro (robot description, xacro)
@@ -4,4 +4,6 @@
     <xacro:include filename="test_lidar.xacro"/>
     <xacro:include filename="wheels.xacro"/>
+    <xacro:include filename="top.xacro"/>
+    <xacro:include filename="realsense_camera.xacro"/>
     <!-- MATERIALS -->
     <material name="white">
@@ -31,4 +33,11 @@
     <link name="base_footprint">
     </link>
+    <joint name="odom" type="fixed">
+        <parent link="base_link"/>
+        <child link="odom_frame"/>
+        <origin xyz="0 0 0" rpy="0 0 0"/>
+    </joint>
+    <link name="odom_frame">
+    </link>
     <!-- CHASSIS LINK -->
     <joint name="chassis_joint" type="fixed">
