Commit message: odom

File: my_bot/description/lidar.xacro (robot description, xacro)
@@ -5,5 +5,5 @@
         <parent link="base_link"/>
         <child link="laser_link"/>
-        <origin xyz="0.15 0 1.34" rpy="0 0 0"/>
+        <origin xyz="0.15 0 1.34" rpy="0 0 1.5708"/>
     </joint>
     <link name="laser_link">

File: my_bot/description/test_lidar.xacro (robot description, xacro)
@@ -23,3 +23,10 @@
         </xacro:inertial_cylinder>
     </link>
+    <joint name="lidar_rotate_joint" type="fixed">
+        <parent link="base_link"/>
+        <child link="lidar_rotate_link"/>
+        <origin xyz="0.2975 -0.012 0.11225" rpy="0 0 0"/>
+    </joint>
+    <link name="lidar_rotate_link">
+    </link>
 </robot>
